File: ETHERTEN2.brd (EAGLE design)
At the start: 68.6 x 53.3 mm, 103 parts, among them IC1 MC33269DT-5.0, IC2 APX811-44UG-7, IC3 ATMEGA16U2-MU, IC4 LM358D, IC5 ATMEGA328P TQFP32, IC6 W5100SQFP80, IC7 MCP24AA025E48, J1 DC_2_1MM, P1 USB-6PSMT, P2 ICSP:MAIN, P3 ICSP:USB, P4 microSD, Q1 FDN340P, Q2 2N7002, Q3 2N7002, U1 HY931147C-RJ45, X1 16MHz, X2 25MHz, X3 16MHz

Commit message: Ethernet chip conversion
Parts:
- removed C17, C25, C26, C28: 100nF, freetronics:0603
- removed IC6: W5100SQFP80, freetronics-marc:SQFP80
- removed R6: 12K3 1%, freetronics:0603
- added IC8: W5500, W5500:W5500
Connections:
- removed net 1V8OUT: C28.1, IC6.33, IC6.69
- removed net N$27: IC6.55, IC6.57, IC6.58, RN7.2
- removed net N$322: IC6.1, R6.2
- net 1V8A: no longer C17.1, IC6.7, IC6.74
- net 1V8_OUT: no longer C26.1, IC6.11, IC6.15, IC6.16
- net 3V3A: no longer IC6.2
- net 3V3D: no longer C25.1, IC6.12, IC6.18, IC6.44, RN7.7
- net COLLED: no longer IC6.71
- net D10_SS: no longer IC6.29
- net D11_MOSI: no longer IC6.28
- net D12_MISO: no longer IC6.27
- net D13_SCK: no longer IC6.30
- net FDXLED: no longer IC6.70
- net GND: no longer C17.2, C25.2, C26.2, C28.2, IC6.10, IC6.13, IC6.14, IC6.17, IC6.19, IC6.20, IC6.21, IC6.22, IC6.23, IC6.24, IC6.25, IC6.26, IC6.32, IC6.34, IC6.35, IC6.36, IC6.37, IC6.38, IC6.39, IC6.4, IC6.40, IC6.41, IC6.42, IC6.43, IC6.45, IC6.46, IC6.47, IC6.48, IC6.49, IC6.50, IC6.51, IC6.52, IC6.53, IC6.54, IC6.63, IC6.64, IC6.65, IC6.68, IC6.77, R6.1
- net INT: no longer IC6.56
- net LINKLED: no longer IC6.66
- net RXIN: no longer IC6.6
- net RXIP: no longer IC6.5
- net SEN: no longer IC6.31
- net SPDLED: no longer IC6.67
- net TXON: no longer IC6.9
- net TXOP: no longer IC6.8
- net WIZRST: no longer IC6.59
- net WRXLED: no longer IC6.72
- net WTXLED: no longer IC6.73
- net XTLN: no longer IC6.75
- net XTLP: no longer IC6.76
Routing:
- net GND: track 187.9 -> 105.6 mm, vias 101 -> 98
- net 1V8A: track 24.2 -> 5.31 mm
- net 1V8OUT: track 17.0 -> 0.00 mm, vias 2 -> 0
- net N$27: track 13.7 -> 0.00 mm
- net N$322: track 6.81 -> 0.00 mm
- net WTXLED: track 17.0 -> 11.9 mm
- net 3V3D: track 181.5 -> 176.7 mm
- net WRXLED: track 15.0 -> 10.5 mm
- net D10_SS: track 54.0 -> 50.1 mm
- net TXOP: track 37.7 -> 33.9 mm
- net COLLED: track 16.2 -> 12.7 mm
- net D13_SCK: track 102.4 -> 98.9 mm
- net TXON: track 40.5 -> 37.1 mm
- net XTLN: track 13.9 -> 10.6 mm
- net WIZRST: track 3.19 -> 0.05 mm
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