File: ETHERUNO.sch (EAGLE design)
At the start: 97 parts, among them IC1 MC33269DT-5.0, IC2 APX811-44UG-7, IC3 ATMEGA16U2-MU, IC4 LM358D, IC5 ATMEGA328P TQFP32, IC7 MCP24AA025E48, J1 DC_2_1MM, J2 USB-C-16P-16P, P2 ICSP:MAIN, P3 ICSP:USB, P4 microSD, Q1 FDN340P, Q2 2N7002, Q3 2N7002, U1 HY931147C-RJ45, X1 16MHz, X2 25MHz, X3 16MHz

Commit message: Added cut-track jumper to isolate D4
Parts:
- added U$8: SJC-NORMAL, SuperHouse-Jumpers:SJC-NORMAL
Connections:
- new net N$27: RN6D.2, U$8.1
- net D4: now also U$8.2; no longer RN6D.2
Other:
- note added: "SKU: EU"
- note added: "SuperHouse EtherUno"
- note added: "V4.0 (2020-05-15)"
- note added: "www.superhouse.tv/etheruno"
- note removed: "Freetronics EtherTen"
- note removed: "SKU: ET"
- note removed: "V3.0 (2013-09-06)"
- note removed: "www.freetronics.com/et"
- moved on the sheet: H1, H4, RN6D

Commit message: Split schematic into separate sheets
Other:
- note added: "Wiznet W6100 Power-On/Reset"
- note removed: "Prototyping Area"
- note removed: "Wiznet W5100 Power-On/Reset"

Commit message: Major rework of schematic to suit W6100
Parts:
- removed C18: 10nF, SuperHouse-DiscreteSemi:CAP0603
- removed IC2: APX811-44UG-7, freetronics-master-v1:APX81X-RESET-IC
- removed LED1: YELLOW, SuperHouse-LEDs:LED0603
- removed Q3: 2N7002, SuperHouse-DiscreteSemi:MOSFET-NCHANNEL-233
- removed R7: 1M 0603, SuperHouse-DiscreteSemi:RESISTOR0603
- removed REG1: LD1117-SOT89, freetronics:V_REG_LM1117SOT89
- removed REG2: LD1117-SOT223, freetronics:V_REG_LM1117SOT223
- removed RN7: 1K, SuperHouse-DiscreteSemi:4R-NCAY16
- removed U$8: SJC-NORMAL, SuperHouse-Jumpers:SJC-NORMAL
- removed X1, X3: 16MHz, SuperHouse-Oscillators:CRYSTALHC49UV
- removed X2: 25MHz, SuperHouse-Oscillators:CRYSTALHC49UV
- added IC6: W6100-LQFP, SuperHouse-ICs:W6100-LQFP
- added L4: 1uH 250mA 0805, SuperHouse-DiscreteSemi:INDUCTOR0805-LARGE
- added SJ7: SJC, SuperHouse-Jumpers:SJC-NORMAL
- added U$17, U$19, U$20: CRYSTAL-GND3X2, SuperHouse-Oscillators:CRYSTAL-GND3X2
- added VR1: LD1117-SOT223, SuperHouse-Regulators:LD1117-SOT223
- added VR2: LD1117-SOT89, SuperHouse-Regulators:LD1117-SOT89
- A6, A7, CD: value M01PTH -> M01; device freetronics-2:M01PTH -> SuperHouse-Connectors:M01-PLAIN
- FID1, FID2, FID3: device freetronics:FIDUCIAL1X2.5 -> SuperHouse-Symbols:FIDUCIAL1X2.5
- IC1: device linear:MC33269D-5.0 -> SuperHouse-Regulators:MC33269-X-5.0-D
- IC3: device freetronics-jon:ATMEL_ATMEGA8U2-MUQFN -> SuperHouse-MCUs:ATMEGA8U2QFN
- L1, L2: device rcl:L-USL2012C -> SuperHouse-DiscreteSemi:INDUCTOR0805-LARGE
- L3: device freetronics-master-v1:INDUCTOR0805-LARGE -> SuperHouse-DiscreteSemi:INDUCTOR0805-LARGE
- R1: value 1M 0603 -> 4K7
- R2: value 27R 0603 -> 4K7
- R3: value 1M -> (none)
- R4, R5: value 22R 0603 -> 22R
- RN1, RN2: value 1K -> 330R
- RN4: device freetronics-master-v1:4R-NCAY16 -> SuperHouse-DiscreteSemi:4R-NCAY16
- SJ1, SJ3: device jumper:SJ -> SuperHouse-Jumpers:SJC-NORMAL
- SJ2: device jumper:SJ -> SuperHouse-Jumpers:SJ-NORMAL
- SJ4: value D2_INT -> (none); device jumper:SJ -> SuperHouse-Jumpers:SJ-NORMAL
- SJ5, SJ6: value SJCN -> SJC; device freetronics-jon:SJCN -> SuperHouse-Jumpers:SJC-NORMAL
Connections:
- removed net 1V8A: C4.+, L1.2
- removed net 1V8_OUT: C3.+, L1.1
- removed net INT: SJ4.2
- removed net N$113: C2.2, IC3.XTAL2, R1.2, X1.2
- removed net N$114: C8.2, R1.1, R2.2, X1.1
- removed net N$330: LED1.C, RN1A.2
- removed net SEN: Q3.D, RN7D.1
- removed net WIZRST: IC2./RESET
- removed net WRXLED: RN1B.1
- removed net WTXLED: RN1A.1
- removed net XTLN: C16.1, R3.2, X2.2
- removed net XTLP: C15.1, R3.1, X2.1
- new net 1V2A: C4.+, IC6.1V2A, L1.2
- new net 1V2D: C3.+, IC6.1V2D, L4.2
- new net 1V2O: IC6.1V2O, L1.1, L4.1
- new net 3.3V: C10.+, IC4A.-IN, IC6.3V3D, L2.1, LED3.A, LED4.A, LED7.A, LED8.A, LED9.A, U1.G+, U1.Y+, VR1.OUT, VR2.OUT
- new net ACTLED: IC6.!ACT, RN1B.1
- new net MODE: IC6.MOD0, R3.2, SJ4.1
- new net N$10: J2.CC2, R1.2
- new net N$30: C15.1, IC6.XSCO, U$17.XTL1
- new net N$31: C2.2, IC3.XTAL2, U$20.XTL1
- new net N$32: C16.1, IC6.XSCI, U$17.XTL2
- new net N$33: IC6.!CS
- new net N$34: J2.CC1, R2.2
- net 3V3A: now also IC6.3V3A; no longer C18.1
- net 3V3D: now also SJ4.2; no longer C10.+, IC4A.-IN, L2.1, LED1.A, LED3.A, LED4.A, LED7.A, LED8.A, LED9.A, REG1.OUT, REG1.OUT@1, REG2.OUT, REG2.OUT@1, RN7D.2, U1.G+, U1.Y+
- net 5V: now also VR1.IN, VR2.IN; no longer IC2.VCC, REG1.IN, REG2.IN
- net COLLED: now also IC6.!COL
- net D10_SS: no longer Q3.G
- net D11_MOSI: now also IC6.MOSI
- net D12_MISO: now also IC6.MISO
- net D13_SCK: now also IC6.SCLK
- net D2: no longer SJ4.1
- net D4: now also SJ7.2; no longer U$8.2
- net FDXLED: now also IC6.!DPX
- net GND: now also IC6.GND, IC6.GNDA, IC6.MOD1, IC6.MOD2, IC6.MOD3, R3.1, U$17.GND, U$17.GND2, U$19.GND, U$19.GND2, U$20.GND, U$20.GND2, VR1.GND, VR2.GND; no longer C18.2, IC2.GND, Q3.S, REG1.ADJ, REG2.ADJ
- net LINKLED: now also IC6.!LINK
- net N$2: now also U$19.XTL1; no longer R7.2, X3.2
- net N$27: now also SJ7.1; no longer U$8.1
- net N$7: now also U$19.XTL2; no longer R7.1, X3.1
- net N$8: now also C8.2, U$20.XTL2; no longer R2.1
- net N$9: now also J2.GND, R1.1, R2.1
- net RESET: now also IC6.!RESET; no longer IC2./MR
- net RXIN: now also IC6.RXIN
- net RXIP: now also IC6.RXIP
- net SPDLED: now also IC6.!SPD
- net TXON: now also IC6.TXON
- net TXOP: now also IC6.TXOP
Other:
- note added: "(C)2020 SuperHouse Automation: www.superhouse.tv"
- note added: "1.2V / 3.3V Decoupling"
- note added: "1V2O is generated by the Wiznet W6100"
- note added: "3V3 800mA Power Supply"
- note added: "5V Power Supply"
- note added: "EtherUno (Arduino compatible with Ethernet)"
- note added: "Ethernet Controller"
- note added: "Ethernet Interface with PoE"
- note added: "ICSP Headers"
- note added: "Licensed under the TAPR Open Hardware License: www.tapr.org/ohl"
- note added: "MAC Address ROM"
- note added: "Micro SD Card Slot"
- note added: "Open: W6100 Closed: W5500"
- note added: "Wiznet Mode Selection"
- note added: "www.superhouse.tv/eu"
- note removed: "1.8V / 3.3V Decoupling"
- note removed: "140ms min, 280ms max"
- note removed: "3V3 Power Supply"
- note removed: "800mA"
- note removed: "< 4.38 Vrst, push-pull output"
- note removed: "<--"
- note removed: "APX811-44UG-7 Reset IC"
- note removed: "DC Regulated Power Supply"
- note removed: "Ethernet Module with PoE"
- note removed: "In Circuit Serial Programming"
- note removed: "SPI D10_SS/nCS low = SEN high = SPI enabled"
- note removed: "SPI MISO tri-state by SS/nCS"
- note removed: "Short across SJ1 GROUND and SJ3 RESET-EN after all other routing"
- note removed: "SuperHouse EtherUno"
- note removed: "Wiznet W6100 Power-On/Reset"
- note removed: "micro SD Card Slot"
- note removed: "www.superhouse.tv/etheruno"

Commit message: Removed ATmega16U2 and added CP2102N for USB-serial conversion
Parts:
- removed C11: 1uF 0603, SuperHouse-DiscreteSemi:CAP0603
- removed C12: 100nF 0603, SuperHouse-DiscreteSemi:CAP0603
- removed C2, C8: 22pF 0603, SuperHouse-DiscreteSemi:CAP0603
- removed IC3: ATMEGA16U2-MU, SuperHouse-MCUs:ATMEGA8U2QFN
- removed P3: ICSP:USB, SuperHouse-Connectors:ICSP-PIN
- removed R4, R5: 22R, SuperHouse-DiscreteSemi:RESISTOR0603
- removed U$20: CRYSTAL-GND3X2, SuperHouse-Oscillators:CRYSTAL-GND3X2
- added C17, C18, C25, C26, C28, C30, C31: 100nF, SuperHouse-DiscreteSemi:CAP0603
- added IC2: CP2102N-A01-GQFN24, SuperHouse-ICs:CP2104
- added R12: 22.1K, SuperHouse-DiscreteSemi:RESISTOR0603
- added R13: 47.5K, SuperHouse-DiscreteSemi:RESISTOR0603
- added R6: 12K 1%, SuperHouse-DiscreteSemi:RESISTOR0603
- added R7: 300R 1%, SuperHouse-DiscreteSemi:RESISTOR0603
- added R9: 10K, SuperHouse-DiscreteSemi:RESISTOR0603
- R1, R2: value 4K7 -> 5K1
- R3: value (none) -> 10K
Connections:
- removed net 3V3D: C29.1, H2.4, P4.VCC, SJ4.2
- removed net D10_SS: H1.3, IC5.PB2(SS/OC1B)
- removed net MISO2: IC3.(MISO)PB3, P3.1
- removed net MOSI2: IC3.(MOSI)PB2, P3.4
- removed net N$117: C11.1, IC3.UCAP
- removed net N$16: J2.D+, R5.2, Z1.1
- removed net N$17: J2.D-, R4.2, Z2.1
- removed net N$31: C2.2, IC3.XTAL2, U$20.XTL1
- removed net N$33: IC6.!CS
- removed net N$8: C8.2, IC3.XTAL1, U$20.XTL2
- removed net RD+: IC3.D+, R5.1
- removed net RD-: IC3.D-, R4.1
- removed net RESET2: IC3.RESET, P3.5, RN4A.1
- removed net RXLED: IC3.PD4, RN3B.2
- removed net SCK2: IC3.(SCLK)PB1, P3.3
- removed net TXLED: IC3.(XCK)PD5, RN3A.2
- new net D+: IC2.D+, J2.D+, Z1.1
- new net D-: IC2.D-, J2.D-, Z2.1
- new net D10_CS: H1.3, IC5.PB2(SS/OC1B), IC6.!CS
- new net N$35: R6.2, R7.1
- new net N$36: IC6.RSET_BG, R6.1
- new net N$37: IC6.!INT, R9.1
- new net N$39: IC2.VBUS, R12.1, R13.2
- new net RX_LED: IC2.GPIO_1, RN3B.2
- new net TX_LED: IC2.GPIO_0, RN3A.2
- net 1V2A: now also C17.1
- net 1V2D: now also C26.1, C28.1, C30.1, C31.1
- net 3.3V: now also C29.1, H2.4, IC2.REGIN, IC2.VDD, IC2.VIO, LED5.A, LED6.A, P4.VCC, R9.2, SJ4.2
- net 3V3A: now also C18.1, C25.1
- net 5V: now also H2.2, R12.2; no longer C12.1, IC3.AVCC, IC3.VCC, LED5.A, LED6.A, P3.2, RN4A.2
- net DTR: now also IC2.DTR; no longer IC3.(CTS)PD7
- net GND: now also C17.2, C18.2, C25.2, C26.2, C28.2, C30.2, C31.2, IC2.GND, IC2.GND_PAD, R13.1, R7.2; no longer C11.2, C12.2, C2.1, C8.1, IC3.GND, IC3.PAD, P3.6, U$20.GND, U$20.GND2
- net USBGND: no longer IC3.UGND
- net USBRXD: now also IC2.TXD; no longer IC3.(TXD1)PD3
- net USBTXD: now also IC2.RXD; no longer IC3.(RXD1)PD2
- net USBVCC: no longer IC3.UVCC
Other:
- note added: "ICSP Header"
- note added: "Open: W6100 (default) Closed: W5500"
- note added: "To power source selection circuit"
- note added: "USB-Serial Converter"
- note removed: "ATmega16U2 Microcontroller"
- note removed: "D2 used if Wiznet Ethernet IC "interrupt" jumper enabled."
- note removed: "ICSP Headers"
- note removed: "Open: W6100 Closed: W5500"
